File: 2-PROJ/23-Carte_Alim_Turbines/23-Carte_Alim_Turbines.kicad_pcb (KiCad board)
At the start: 2 copper layers, 80 x 40 mm, 48 parts, among them J1 Conn_01x03, J2 Conn_01x03, J3 Conn_01x03, J4 Conn_01x03, Q1 2N7002, Q2 SUM110P06-08L, Q3 SUM110P06-08L, Q4 SUM110P06-08L, Q5 SUM110P06-08L, Q6 2N7002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

Commit message: Work in progress
Parts:
- moved F2 3.84 mm to (122.7, 79.4), turned to -90 degrees
- moved F1 3.74 mm to (122.7, 60.5), turned to 90 degrees
- moved C6 3.50 mm to (86.1, 75.0), turned to -90 degrees
- moved C2 3.50 mm to (86.1, 65.0), turned to 90 degrees
- moved R18 1.18 mm to (74.5, 73.3), turned to 90 degrees
Connections:
- U1 pad 1: /5P -> Net-(R3-Pad2)
- U1 pad 2: Net-(R3-Pad2) -> /5P
Routing:
- net Net-(Q1-D): track 0.00 -> 54.8 mm
- net GND: track 0.00 -> 46.9 mm, vias 0 -> 1
- net Net-(D1-A): track 0.00 -> 31.9 mm
- net /5P: track 0.00 -> 30.5 mm
- net Net-(D3-A): track 0.00 -> 26.2 mm
- net /5V_ESC_T2: track 0.00 -> 21.8 mm
- net /5V_ESC_T1: track 0.00 -> 20.4 mm
- net Net-(J2-Pin_3): track 0.00 -> 17.0 mm
- net Net-(J1-Pin_3): track 0.00 -> 13.7 mm
- net /SW_AU: track 0.00 -> 5.58 mm, vias 0 -> 1
- net Net-(Q1-G): track 0.00 -> 5.00 mm
- net Net-(J4-Pin_3): track 0.00 -> 4.28 mm
- net Net-(J3-Pin_3): track 0.00 -> 4.14 mm
- net Net-(C8-Pad1): track 0.00 -> 3.49 mm
- net Net-(Q6-G): track 0.00 -> 3.47 mm
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- added copper zone on B.Cu, net /PWR_T1
- added copper zone on F.Cu, net /PWR_T1
- added copper zone on B.Cu, net /PWR_T2
- added copper zone on F.Cu, net /PWR_T2
- added copper zone on B.Cu, net /VBATT_24V_T1
- added copper zone on F.Cu, net /VBATT_24V_T1
- added copper zone on B.Cu, net /VBATT_24V_T2
- added copper zone on F.Cu, net /VBATT_24V_T2
- added copper zone on B.Cu, net GNDPWR
- added copper zone on F.Cu, net GNDPWR
