File: 2-PROJ/23-Carte_Alim_Turbines/23-Carte_Alim_Turbines.kicad_sch (KiCad schematic)
At the start: 60 parts, among them J1 Conn_01x03, J2 Conn_01x03, J3 Conn_01x03, J4 Conn_01x03, Q1 2N7002, Q2 SUM110P06-08L, Q3 SUM110P06-08L, Q4 SUM110P06-08L, Q5 SUM110P06-08L, Q6 2N7002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

Commit message: petite correction avant generation du dossier
Parts:
- added H5, H6: MountingHole, MountingHole:MountingHole_2mm, symbol Mechanical:MountingHole
- H1, H2, H3, H4, W1, W2, W3, W4, W5, W6: now left out of the parts list
Changed lines of the file:
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@@
   )
   (symbol (lib_id "Mechanical:MountingHole_Pad") (at 125.73 24.13 90) (unit 1)
-    (in_bom yes) (on_board yes) (dnp no)
+    (in_bom no) (on_board yes) (dnp no)
     (property "Reference" "W1" (at 120.65 24.13 90)
       (effects (font (size 1.27 1.27)))
@@
   )
   (symbol (lib_name "MountingHole_Pad_3") (lib_id "Mechanical:MountingHole_Pad") (at 264.16 152.4 0) (unit 1)
-    (in_bom yes) (on_board yes) (dnp no) (fields_autoplaced)
+    (in_bom no) (on_board yes) (dnp no) (fields_autoplaced)
     (property "Reference" "H4" (at 266.7 149.86 0)
       (effects (font (size 1.27 1.27)) (justify left))
@@
   )
   (symbol (lib_name "MountingHole_Pad_1") (lib_id "Mechanical:MountingHole_Pad") (at 223.52 152.4 0) (unit 1)
-    (in_bom yes) (on_board yes) (dnp no) (fields_autoplaced)
+    (in_bom no) (on_board yes) (dnp no) (fields_autoplaced)
     (property "Reference" "H2" (at 226.06 149.86 0)
       (effects (font (size 1.27 1.27)) (justify left))
@@
     )
   )
+  (symbol (lib_id "Mechanical:MountingHole") (at 223.52 142.24 0) (unit 1)
+    (in_bom no) (on_board yes) (dnp no) (fields_autoplaced)
+    (property "Reference" "H6" (at 226.06 140.97 0)
+      (effects (font (size 1.27 1.27)) (justify left))
+    )
+    (property "Value" "MountingHole" (at 226.06 143.51 0)
+      (effects (font (size 1.27 1.27)) (justify left))
+    )
+    (property "Footprint" "MountingHole:MountingHole_2mm" (at 223.52 142.24 0)
+      (effects (font (size 1.27 1.27)) hide)
+    )
+    (property "Datasheet" "~" (at 223.52 142.24 0)
+      (effects (font (size 1.27 1.27)) hide)
+    )
+    (instances
+      (project "23-Carte_Alim_Turbines"
+        (path "/cdcb0d26-1eaa-4cdc-8d62-f877abffbd60"
+          (reference "H6") (unit 1)
+        )
+      )
+    )
+  )
   (symbol (lib_id "Device:R") (at 64.77 125.73 0) (unit 1)
     (in_bom yes) (on_board yes) (dnp no)
@@
   )
   (symbol (lib_name "MountingHole_Pad_4") (lib_id "Mechanical:MountingHole_Pad") (at 243.84 152.4 0) (unit 1)
-    (in_bom yes) (on_board yes) (dnp no) (fields_autoplaced)
+    (in_bom no) (on_board yes) (dnp no) (fields_autoplaced)
     (property "Reference" "H3" (at 246.38 149.86 0)
       (effects (font (size 1.27 1.27)) (justify left))
@@
   )
   (symbol (lib_id "Mechanical:MountingHole_Pad") (at 260.35 41.91 270) (unit 1)
-    (in_bom yes) (on_board yes) (dnp no)
+    (in_bom no) (on_board yes) (dnp no)
     (property "Reference" "W4" (at 264.16 41.91 90)
       (effects (font (size 1.27 1.27)) (justify left))
@@
     )
   )
+  (symbol (lib_id "Mechanical:MountingHole") (at 203.2 142.24 0) (unit 1)
+    (in_bom no) (on_board yes) (dnp no) (fields_autoplaced)
+    (property "Reference" "H5" (at 205.74 140.97 0)
+      (effects (font (size 1.27 1.27)) (justify left))
+    )
+    (property "Value" "MountingHole" (at 205.74 143.51 0)
+      (effects (font (size 1.27 1.27)) (justify left))
+    )
+    (property "Footprint" "MountingHole:MountingHole_2mm" (at 203.2 142.24 0)
+      (effects (font (size 1.27 1.27)) hide)
+    )
+    (property "Datasheet" "~" (at 203.2 142.24 0)
+      (effects (font (size 1.27 1.27)) hide)
+    )
+    (instances
+      (project "23-Carte_Alim_Turbines"
+        (path "/cdcb0d26-1eaa-4cdc-8d62-f877abffbd60"
+          (reference "H5") (unit 1)
+        )
+      )
+    )
+  )
   (symbol (lib_id "power:GND") (at 38.1 163.83 0) (unit 1)
     (in_bom yes) (on_board yes) (dnp no) (fields_autoplaced)
@@
   )
   (symbol (lib_id "Mechanical:MountingHole_Pad") (at 260.35 34.29 270) (unit 1)
-    (in_bom yes) (on_board yes) (dnp no)
+    (in_bom no) (on_board yes) (dnp no)
     (property "Reference" "W3" (at 264.16 34.29 90)
       (effects (font (size 1.27 1.27)) (justify left))
@@
   )
   (symbol (lib_name "MountingHole_Pad_2") (lib_id "Mechanical:MountingHole_Pad") (at 203.2 152.4 0) (unit 1)
-    (in_bom yes) (on_board yes) (dnp no) (fields_autoplaced)
+    (in_bom no) (on_board yes) (dnp no) (fields_autoplaced)
     (property "Reference" "H1" (at 205.74 149.86 0)
       (effects (font (size 1.27 1.27)) (justify left))
@@
   )
   (symbol (lib_id "Mechanical:MountingHole_Pad") (at 260.35 78.74 270) (unit 1)
-    (in_bom yes) (on_board yes) (dnp no)
+    (in_bom no) (on_board yes) (dnp no)
     (property "Reference" "W6" (at 264.16 78.74 90)
       (effects (font (size 1.27 1.27)) (justify left))
@@
   )
   (symbol (lib_id "Mechanical:MountingHole_Pad") (at 260.35 71.12 270) (unit 1)
-    (in_bom yes) (on_board yes) (dnp no)
+    (in_bom no) (on_board yes) (dnp no)
     (property "Reference" "W5" (at 264.16 71.12 90)
       (effects (font (size 1.27 1.27)) (justify left))
@@
   )
   (symbol (lib_id "Mechanical:MountingHole_Pad") (at 125.73 34.29 90) (unit 1)
-    (in_bom yes) (on_board yes) (dnp no)
+    (in_bom no) (on_board yes) (dnp no)
     (property "Reference" "W2" (at 120.65 34.29 90)
       (effects (font (size 1.27 1.27)))

Commit message: generation des fichiers de fabrication des cartes
Parts:
- R10, R18: value R -> 10k
- R11, R13: value R -> 22
- R12, R3, R4: value R -> 330
- R15, R16, R17: value R -> 1k
Changed lines of the file:
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@@
-    (effects (font (size 1.27 1.27)) (justify left bottom))
-  )
-  (label "5P" (at 64.77 137.16 0) (fields_autoplaced)
     (effects (font (size 1.27 1.27)) (justify left bottom))
   )
@@
   (symbol (lib_id "Device:R") (at 106.68 116.84 0) (unit 1)
     (in_bom yes) (on_board yes) (dnp no) (fields_autoplaced)
-    (property "Reference" "R10" (at 109.22 116.205 0)
-      (effects (font (size 1.27 1.27)) (justify left))
-    )
-    (property "Value" "R" (at 109.22 118.745 0)
+    (property "Reference" "R10" (at 109.22 115.57 0)
+      (effects (font (size 1.27 1.27)) (justify left))
+    )
+    (property "Value" "10k" (at 109.22 118.11 0)
       (effects (font (size 1.27 1.27)) (justify left))
     )
@@
       (effects (font (size 1.27 1.27)))
     )
-    (property "Value" "R" (at 81.28 146.05 90)
+    (property "Value" "330" (at 81.28 146.05 90)
       (effects (font (size 1.27 1.27)))
     )
@@
       (effects (font (size 1.27 1.27)) (justify right))
     )
-    (property "Value" "100k" (at 63.5 123.19 0)
+    (property "Value" "100k" (at 62.23 128.27 0)
       (effects (font (size 1.27 1.27)) (justify right))
     )
@@
       (effects (font (size 1.27 1.27)))
     )
-    (property "Value" "R" (at 55.88 153.67 90)
+    (property "Value" "22" (at 55.88 153.67 90)
       (effects (font (size 1.27 1.27)))
     )
@@
       (effects (font (size 1.27 1.27)))
     )
-    (property "Value" "R" (at 81.28 111.76 90)
+    (property "Value" "330" (at 86.36 109.22 90)
       (effects (font (size 1.27 1.27)))
     )
@@
       (effects (font (size 1.27 1.27)) (justify right))
     )
-    (property "Value" "100k" (at 63.5 153.67 0)
+    (property "Value" "100k" (at 62.23 158.75 0)
       (effects (font (size 1.27 1.27)) (justify right))
     )
@@
   (symbol (lib_id "Device:R") (at 106.68 146.05 0) (unit 1)
     (in_bom yes) (on_board yes) (dnp no) (fields_autoplaced)
-    (property "Reference" "R18" (at 109.22 145.415 0)
-      (effects (font (size 1.27 1.27)) (justify left))
-    )
-    (property "Value" "R" (at 109.22 147.955 0)
+    (property "Reference" "R18" (at 109.22 144.78 0)
+      (effects (font (size 1.27 1.27)) (justify left))
+    )
+    (property "Value" "10k" (at 109.22 147.32 0)
       (effects (font (size 1.27 1.27)) (justify left))
     )
@@
       (effects (font (size 1.27 1.27)))
     )
-    (property "Value" "R" (at 48.26 133.35 0)
+    (property "Value" "1k" (at 48.26 133.35 0)
       (effects (font (size 1.27 1.27)))
     )
@@
       (effects (font (size 1.27 1.27)))
     )
-    (property "Value" "R" (at 146.05 130.81 90)
+    (property "Value" "1k" (at 146.05 130.81 90)
       (effects (font (size 1.27 1.27)))
     )
@@
       (effects (font (size 1.27 1.27)))
     )
-    (property "Value" "R" (at 81.28 69.85 90)
+    (property "Value" "330" (at 81.28 69.85 90)
       (effects (font (size 1.27 1.27)))
     )
@@
       (effects (font (size 1.27 1.27)))
     )
-    (property "Value" "R" (at 55.88 123.19 90)
+    (property "Value" "22" (at 55.88 123.19 90)
       (effects (font (size 1.27 1.27)))
     )
@@
       (effects (font (size 1.27 1.27)))
     )
-    (property "Value" "R" (at 146.05 119.38 90)
-      (effects (font (size 1.27 1.27)))
-    )
+    (property "Value" "1k" (at 146.05 119.38 90)
+      (effects (font (size 1.27 1.27)))
+    )
