File: 2-PROJ/24-Carte_Mere_PAMI_2024/CAN.kicad_sch (KiCad schematic)
At the start: 10 parts, among them U3 MCP2515-xST, U4 MCP2551-I-SN, Y1 16 MHz

Commit message: Carte Mère PAMI - Work In Progress
Parts:
- added R7: 120, Resistor_SMD:R_0603_1608Metric_Pad0.98x0.95mm_HandSolder, symbol Device:R
Connections:
- net CANH: now also R7.2
- net CANL: now also R7.1
- net at C1.1, U3.9 (OSC1): now also Y1.1; no longer Y1.2
- net at C1.1, U3.8 (OSC2): now also Y1.2; no longer Y1.1
Other:
- moved on the sheet: Y1
Changed lines of the file:
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@@
   (junction (at 96.52 38.1) (diameter 0) (color 0 0 0 0)
   )
+  (junction (at 193.04 73.66) (diameter 0) (color 0 0 0 0)
+  )
   (junction (at 71.12 95.25) (diameter 0) (color 0 0 0 0)
+  )
+  (junction (at 180.34 68.58) (diameter 0) (color 0 0 0 0)
   )
   (no_connect (at 111.76 88.9))
@@
     (stroke (width 0) (type default))
   )
-  (wire (pts (xy 171.45 68.58) (xy 179.07 68.58))
+  (wire (pts (xy 171.45 68.58) (xy 180.34 68.58))
+    (stroke (width 0) (type default))
+  )
+  (wire (pts (xy 190.5 71.12) (xy 193.04 71.12))
     (stroke (width 0) (type default))
   )
@@
     (stroke (width 0) (type default))
   )
+  (wire (pts (xy 193.04 71.12) (xy 193.04 73.66))
+    (stroke (width 0) (type default))
+  )
   (wire (pts (xy 63.5 110.49) (xy 71.12 110.49))
     (stroke (width 0) (type default))
   )
+  (wire (pts (xy 193.04 73.66) (xy 207.01 73.66))
+    (stroke (width 0) (type default))
+  )
   (wire (pts (xy 96.52 38.1) (xy 96.52 60.96))
     (stroke (width 0) (type default))
@@
     (stroke (width 0) (type default))
   )
-  (wire (pts (xy 171.45 73.66) (xy 179.07 73.66))
+  (wire (pts (xy 171.45 73.66) (xy 193.04 73.66))
     (stroke (width 0) (type default))
   )
@@
     (stroke (width 0) (type default))
   )
+  (wire (pts (xy 182.88 71.12) (xy 180.34 71.12))
+    (stroke (width 0) (type default))
+  )
   (wire (pts (xy 140.97 60.96) (xy 140.97 76.2))
     (stroke (width 0) (type default))
@@
   )
   (wire (pts (xy 128.27 66.04) (xy 130.81 68.58))
+    (stroke (width 0) (type default))
+  )
+  (wire (pts (xy 180.34 68.58) (xy 207.01 68.58))
+    (stroke (width 0) (type default))
+  )
+  (wire (pts (xy 180.34 71.12) (xy 180.34 68.58))
     (stroke (width 0) (type default))
   )
@@
     (effects (font (size 1.27 1.27)) (justify right))
   )
-  (hierarchical_label "CANH" (shape bidirectional) (at 179.07 68.58 0) (fields_autoplaced)
+  (hierarchical_label "CANH" (shape bidirectional) (at 207.01 68.58 0) (fields_autoplaced)
     (effects (font (size 1.27 1.27)) (justify left))
   )
@@
     (effects (font (size 1.27 1.27)) (justify right))
   )
-  (hierarchical_label "CANL" (shape bidirectional) (at 179.07 73.66 0) (fields_autoplaced)
+  (hierarchical_label "CANL" (shape bidirectional) (at 207.01 73.66 0) (fields_autoplaced)
     (effects (font (size 1.27 1.27)) (justify left))
   )
@@
     )
   )
-  (symbol (lib_id "Device:Crystal") (at 63.5 95.25 0) (unit 1)
+  (symbol (lib_id "Device:Crystal") (at 63.5 95.25 180) (unit 1)
     (in_bom yes) (on_board yes) (dnp no) (fields_autoplaced)
     (property "Reference" "Y1" (at 63.5 88.9 0)
@@
         )
       )
+    )
+  )
+  (symbol (lib_id "Device:R") (at 186.69 71.12 270) (unit 1)
+    (in_bom yes) (on_board yes) (dnp no)
+    (property "Reference" "R7" (at 186.69 74.93 90)
+      (effects (font (size 1.27 1.27)) (justify right))
+    )
+    (property "Value" "120" (at 186.69 77.47 90)
+      (effects (font (size 1.27 1.27)) (justify right))
+    )
+    (property "Footprint" "Resistor_SMD:R_0603_1608Metric_Pad0.98x0.95mm_HandSolder" (at 186.69 69.342 90)
+      (effects (font (size 1.27 1.27)) hide)
+    )
+    (property "Datasheet" "~" (at 186.69 71.12 0)
+      (effects (font (size 1.27 1.27)) hide)
+    )
+    (pin "1")
+    (pin "2")
+    (instances
+      (project "PAMI_Mainboard_2024_v1"
+        (path "/71a486c7-371a-4a12-ac74-c4a4c1234df0"
+          (reference "R7") (unit 1)
+        )
+        (path "/71a486c7-371a-4a12-ac74-c4a4c1234df0/8c56106a-6f80-41c5-8219-56e120df5552"
+          (reference "R15") (unit 1)
+        )
+        (path "/71a486c7-371a-4a12-ac74-c4a4c1234df0/921d2156-3b7a-47e8-98e0-dba8d6261338"
+          (reference "R6") (unit 1)
+        )
+      )

Commit message: CM PAMI 2024 - WIP
Parts:
- R1, R7: now not fitted; now left out of the parts list
Changed lines of the file:
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@@
     (effects (font (size 1.27 1.27)) (justify left))
   )
-  (hierarchical_label "INT" (shape input) (at 121.92 81.28 0) (fields_autoplaced)
+  (hierarchical_label "INT" (shape output) (at 121.92 81.28 0) (fields_autoplaced)
     (effects (font (size 1.27 1.27)) (justify left))
   )
@@
   )
   (symbol (lib_id "Device:R") (at 140.97 57.15 180) (unit 1)
-    (in_bom yes) (on_board yes) (dnp no) (fields_autoplaced)
+    (in_bom no) (on_board yes) (dnp yes) (fields_autoplaced)
     (property "Reference" "R1" (at 143.51 56.515 0)
       (effects (font (size 1.27 1.27)) (justify right))
@@
   )
   (symbol (lib_id "Device:R") (at 186.69 71.12 270) (unit 1)
-    (in_bom yes) (on_board yes) (dnp no)
+    (in_bom no) (on_board yes) (dnp yes)
     (property "Reference" "R7" (at 186.69 74.93 90)
       (effects (font (size 1.27 1.27)) (justify right))
@@
   )
   (symbol (lib_id "Device:R") (at 140.97 83.82 180) (unit 1)
-    (in_bom yes) (on_board yes) (dnp no)
+    (in_bom no) (on_board yes) (dnp yes)
     (property "Reference" "R1" (at 143.51 83.82 90)
       (effects (font (size 1.27 1.27)))
