File: 2-PROJ/24-Carte_Mere_PAMI_2024/SX1509.kicad_sch (KiCad schematic)
At the start: 8 parts

Commit message: Carte Mère PAMI - Work In Progress
Parts:
- added J7 (x16): Conn_01x03, Connector_PinHeader_2.54mm:PinHeader_1x03_P2.54mm_Vertical, symbol Connector_Generic:Conn_01x03
Connections:
- net GND: now also J7.1 (Pin_1), J7.1 (Pin_1), J7.1 (Pin_1), J7.1 (Pin_1), J7.1 (Pin_1), J7.1 (Pin_1), J7.1 (Pin_1), J7.1 (Pin_1), J7.1 (Pin_1), J7.1 (Pin_1), J7.1 (Pin_1), J7.1 (Pin_1), J7.1 (Pin_1), J7.1 (Pin_1), J7.1 (Pin_1), J7.1 (Pin_1)
- net SX_IO_0: now also J7.3 (Pin_3)
- net SX_IO_1: now also J7.3 (Pin_3)
- net SX_IO_10: now also J7.3 (Pin_3)
- net SX_IO_11: now also J7.3 (Pin_3)
- net SX_IO_12: now also J7.3 (Pin_3)
- net SX_IO_13: now also J7.3 (Pin_3)
- net SX_IO_14: now also J7.3 (Pin_3)
- net SX_IO_15: now also J7.3 (Pin_3)
- net SX_IO_2: now also J7.3 (Pin_3)
- net SX_IO_3: now also J7.3 (Pin_3)
- net SX_IO_4: now also J7.3 (Pin_3)
- net SX_IO_5: now also J7.3 (Pin_3)
- net SX_IO_6: now also J7.3 (Pin_3)
- net SX_IO_7: now also J7.3 (Pin_3)
- net SX_IO_8: now also J7.3 (Pin_3)
- net SX_IO_9: now also J7.3 (Pin_3)
- new net +5P: J7.2 (Pin_2), J7.2 (Pin_2), J7.2 (Pin_2), J7.2 (Pin_2), J7.2 (Pin_2), J7.2 (Pin_2), J7.2 (Pin_2), J7.2 (Pin_2), J7.2 (Pin_2), J7.2 (Pin_2), J7.2 (Pin_2), J7.2 (Pin_2), J7.2 (Pin_2), J7.2 (Pin_2), J7.2 (Pin_2), J7.2 (Pin_2)
Other:
- moved on the sheet: C1, U1

Commit message: CM PAMI 2024 - WIP
Parts:
- added C8 (x2): 470uF, Capacitor_THT:C_Radial_D8.0mm_H11.5mm_P3.50mm, symbol Device:C_Polarized_Small
Connections:
- net +5P: now also C8.1, C8.1
- net GND: now also C8.2, C8.2
Other:
- note added: "Ajouter resistances en serie sur toutes les GPIO"
- note added: "Les SX150x ont des pull-up / pull-down internes"
Changed lines of the file:
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@@
   (junction (at 152.4 63.5) (diameter 0) (color 0 0 0 0)
   )
+  (junction (at 72.39 38.1) (diameter 0) (color 0 0 0 0)
+  )
   (junction (at 152.4 119.38) (diameter 0) (color 0 0 0 0)
   )
+  (junction (at 220.98 43.18) (diameter 0) (color 0 0 0 0)
+  )
   (junction (at 152.4 44.45) (diameter 0) (color 0 0 0 0)
   )
@@
   (junction (at 74.93 104.14) (diameter 0) (color 0 0 0 0)
   )
+  (junction (at 223.52 38.1) (diameter 0) (color 0 0 0 0)
+  )
   (junction (at 127 105.41) (diameter 0) (color 0 0 0 0)
   )
@@
   )
   (junction (at 220.98 114.3) (diameter 0) (color 0 0 0 0)
+  )
+  (junction (at 74.93 43.18) (diameter 0) (color 0 0 0 0)
   )
   (junction (at 52.07 160.02) (diameter 0) (color 0 0 0 0)
@@
     (stroke (width 0) (type default))
   )
-  (wire (pts (xy 223.52 45.72) (xy 223.52 36.83))
+  (wire (pts (xy 223.52 45.72) (xy 223.52 38.1))
     (stroke (width 0) (type default))
   )
@@
     (stroke (width 0) (type default))
   )
+  (wire (pts (xy 215.9 38.1) (xy 223.52 38.1))
+    (stroke (width 0) (type default))
+  )
   (wire (pts (xy 227.33 78.74) (xy 209.55 78.74))
     (stroke (width 0) (type default))
@@
     (stroke (width 0) (type default))
   )
+  (wire (pts (xy 72.39 38.1) (xy 81.28 38.1))
+    (stroke (width 0) (type default))
+  )
   (wire (pts (xy 67.31 170.18) (xy 67.31 181.61))
     (stroke (width 0) (type default))
@@
     (stroke (width 0) (type default))
   )
+  (wire (pts (xy 72.39 38.1) (xy 72.39 36.83))
+    (stroke (width 0) (type default))
+  )
   (wire (pts (xy 132.08 107.95) (xy 107.95 107.95))
     (stroke (width 0) (type default))
@@
     (stroke (width 0) (type default))
   )
-  (wire (pts (xy 72.39 45.72) (xy 72.39 36.83))
+  (wire (pts (xy 72.39 45.72) (xy 72.39 38.1))
     (stroke (width 0) (type default))
   )
@@
     (stroke (width 0) (type default))
   )
+  (wire (pts (xy 215.9 43.18) (xy 220.98 43.18))
+    (stroke (width 0) (type default))
+  )
   (wire (pts (xy 52.07 160.02) (xy 52.07 162.56))
     (stroke (width 0) (type default))
@@
     (stroke (width 0) (type default))
   )
+  (wire (pts (xy 223.52 38.1) (xy 223.52 36.83))
+    (stroke (width 0) (type default))
+  )
   (wire (pts (xy 173.99 77.47) (xy 204.47 77.47))
     (stroke (width 0) (type default))
@@
   )
   (wire (pts (xy 74.93 53.34) (xy 74.93 63.5))
+    (stroke (width 0) (type default))
+  )
+  (wire (pts (xy 74.93 43.18) (xy 81.28 43.18))
     (stroke (width 0) (type default))
   )
@@
     (effects (font (size 1.27 1.27)) (justify left bottom))
   )
+  (text "Ajouter resistances en serie sur toutes les GPIO" (at 64.77 -8.89 0)
+    (effects (font (size 1.27 1.27)) (justify left bottom))
+  )
   (text "Assignation des I/O SX1509:\n- 6 servos (max 8)\n- 4 entrées \"pare-chocs\"\n- 2 capteurs TOR (nécessite une pull-down)\n=> Disons 8 capteurs + 8 servos\n\nLe capteur de position aura aussi une IT.\n"
     (at 198.12 156.21 0)
+    (effects (font (size 1.27 1.27)) (justify left bottom))
+  )
+  (text "Les SX150x ont des pull-up / pull-down internes" (at 196.85 138.43 0)
     (effects (font (size 1.27 1.27)) (justify left bottom))
   )
@@
     )
   )
+  (symbol (lib_id "Device:C_Polarized_Small") (at 81.28 40.64 0) (unit 1)
+    (in_bom yes) (on_board yes) (dnp no)
+    (property "Reference" "C8" (at 87.63 39.37 0)
+      (effects (font (size 1.27 1.27)) (justify left))
+    )
+    (property "Value" "470uF" (at 86.36 41.91 0)
+      (effects (font (size 1.27 1.27)) (justify left))
+    )
+    (property "Footprint" "Capacitor_THT:C_Radial_D8.0mm_H11.5mm_P3.50mm" (at 81.28 40.64 0)
+      (effects (font (size 1.27 1.27)) hide)
+    )
+    (property "Datasheet" "~" (at 81.28 40.64 0)
+      (effects (font (size 1.27 1.27)) hide)
+    )
+    (pin "1")
+    (pin "2")
+    (instances
+      (project "PAMI_Mainboard_2024_v1"
+        (path "/71a486c7-371a-4a12-ac74-c4a4c1234df0"
+          (reference "C8") (unit 1)
+        )
+        (path "/71a486c7-371a-4a12-ac74-c4a4c1234df0/921d2156-3b7a-47e8-98e0-dba8d6261338"
+          (reference "C10") (unit 1)
+        )
+      )
+      (project "23-Carte_Alim_Turbines"
+        (path "/cdcb0d26-1eaa-4cdc-8d62-f877abffbd60"
+          (reference "C2") (unit 1)
+        )
+      )
+    )
+  )
   (symbol (lib_id "Connector_Generic:Conn_01x03") (at 63.5 106.68 0) (mirror y) (unit 1)
     (in_bom yes) (on_board yes) (dnp no) (fields_autoplaced)
@@
         )
       )
+    )
+  )
+  (symbol (lib_id "Device:C_Polarized_Small") (at 215.9 40.64 0) (unit 1)
+    (in_bom yes) (on_board yes) (dnp no)
+    (property "Reference" "C8" (at 208.28 39.37 0)
+      (effects (font (size 1.27 1.27)) (justify left))
+    )
+    (property "Value" "470uF" (at 207.01 41.91 0)
+      (effects (font (size 1.27 1.27)) (justify left))
+    )
+    (property "Footprint" "Capacitor_THT:C_Radial_D8.0mm_H11.5mm_P3.50mm" (at 215.9 40.64 0)
+      (effects (font (size 1.27 1.27)) hide)
+    )
+    (property "Datasheet" "~" (at 215.9 40.64 0)
+      (effects (font (size 1.27 1.27)) hide)
+    )
+    (pin "1")
+    (pin "2")
+    (instances
+      (project "PAMI_Mainboard_2024_v1"
+        (path "/71a486c7-371a-4a12-ac74-c4a4c1234df0"
+          (reference "C8") (unit 1)
+        )
+        (path "/71a486c7-371a-4a12-ac74-c4a4c1234df0/921d2156-3b7a-47e8-98e0-dba8d6261338"
+          (reference "C9") (unit 1)
+        )
+      )
+      (project "23-Carte_Alim_Turbines"
+        (path "/cdcb0d26-1eaa-4cdc-8d62-f877abffbd60"
+          (reference "C2") (unit 1)
+        )
+      )

Commit message: CM PAMI 2024 - WIP
Parts:
- added R13 (x16): 1K, Resistor_SMD:R_0603_1608Metric_Pad0.98x0.95mm_HandSolder, symbol Device:R
Connections:
- net SX_IO_0: now also R13.1; no longer J7.3 (Pin_3)
- net SX_IO_1: now also R13.1; no longer J7.3 (Pin_3)
- net SX_IO_10: now also R13.2; no longer J7.3 (Pin_3)
- net SX_IO_11: now also R13.2; no longer J7.3 (Pin_3)
- net SX_IO_12: now also R13.2; no longer J7.3 (Pin_3)
- net SX_IO_13: now also R13.2; no longer J7.3 (Pin_3)
- net SX_IO_14: now also R13.2; no longer J7.3 (Pin_3)
- net SX_IO_15: now also R13.2; no longer J7.3 (Pin_3)
- net SX_IO_2: now also R13.1; no longer J7.3 (Pin_3)
- net SX_IO_3: now also R13.1; no longer J7.3 (Pin_3)
- net SX_IO_4: now also R13.1; no longer J7.3 (Pin_3)
- net SX_IO_5: now also R13.1; no longer J7.3 (Pin_3)
- net SX_IO_6: now also R13.1; no longer J7.3 (Pin_3)
- net SX_IO_7: now also R13.1; no longer J7.3 (Pin_3)
- net SX_IO_8: now also R13.2; no longer J7.3 (Pin_3)
- net SX_IO_9: now also R13.2; no longer J7.3 (Pin_3)
- new net: J7.3 (Pin_3), R13.1 (x8)
- new net: J7.3 (Pin_3), R13.2 (x8)
