File: 2-PROJ/27-Carte_Mere_PAMI_2025/Carte_Mere_PAMI_2025.kicad_sch (KiCad schematic)
At the start: 109 parts, among them J1 Conn_01x03, J10 Conn_01x04, J11 Conn_01x03, J12 Conn_01x03, J13 Conn_01x03, J14 Conn_01x03, J15 3.5mm WR-TBL, J16 Conn_01x04, J17 Conn_01x02, J18 Conn_01x02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

Commit message: préplacement carte PAMI 2025
Parts:
- C22: footprint Capacitor_THT:C_Radial_D8.0mm_H11.5mm_P3.50mm -> Capacitor_THT:C_Radial_D6.3mm_H11.0mm_P2.50mm
- J15, J7: value 3.5mm WR-TBL -> Conn_01x02; footprint ConnectorsEvo:691321100002 -> Connector_Wire:SolderWire-0.75sqmm_1x02_P4.8mm_D1.25mm_OD2.3mm; symbol Connector:Screw_Terminal_01x02 -> Connector_Generic:Conn_01x02
- J17, J18, J19, J3: footprint Connector_PinHeader_2.54mm:PinHeader_1x03_P2.54mm_Vertical -> Connector_PinHeader_2.54mm:PinHeader_1x02_P2.54mm_Vertical
- J8: footprint Connector_PinHeader_2.54mm:PinHeader_1x04_P2.54mm_Vertical -> Carte_Mere_PAMI_2025:Ecran_OLED0.9_Waveshare
- SW1: footprint Connector_PinHeader_2.54mm:PinHeader_1x03_P2.54mm_Vertical -> SW_Slide_SPDT_Straight_CK_OS102011MS2Q
Connections:
- net +5L: now also J2.1 (Pin_1); no longer J2.8 (Pin_8)
- net +5P: now also J2.4 (Pin_4), J3.2 (Pin_2), R1.2; no longer D1.2 (A), J2.5 (Pin_5), J3.1 (Pin_1)
- net ALIM_EN_5L: now also J2.8 (Pin_8), SW1.1 (C); no longer J2.1 (Pin_1), SW1.3 (A)
- net CaptTOR_1: now also J2.5 (Pin_5); no longer J2.4 (Pin_4)
- net CaptTOR_2: now also J2.6 (Pin_6); no longer J2.3 (Pin_3)
- net EN_5L: now also J2.7 (Pin_7), SW1.3 (A); no longer J2.2 (Pin_2)
- net GND: now also D1.1 (K), J17.1 (Pin_1), J18.1 (Pin_1), J19.1 (Pin_1), J2.2 (Pin_2), J2.3 (Pin_3); no longer J17.2 (Pin_2), J18.2 (Pin_2), J19.2 (Pin_2), J2.6 (Pin_6), J2.7 (Pin_7), R1.1
- net uSW1: now also J17.2 (Pin_2); no longer J17.1 (Pin_1)
- net uSW2: now also J18.2 (Pin_2); no longer J18.1 (Pin_1)
- net uSW3: now also J19.2 (Pin_2); no longer J19.1 (Pin_1)
- net at C6.2, D2.2 (A), Q1.3 (D): now also J3.1 (Pin_1); no longer J3.2 (Pin_2)
- new net: D1.2 (A), R1.1
Other:
- moved on the sheet: D1, R1

Commit message: WIP routage avec ajout d'un AU_STATUS à la place de la LED statut
Parts:
- removed D4: LED, LED_SMD:LED_0603_1608Metric, symbol Device:LED
- added C29: 100nF, Capacitor_SMD:C_0603_1608Metric_Pad1.08x0.95mm_HandSolder, symbol Device:C
- added R26: 10k, Resistor_SMD:R_0603_1608Metric_Pad0.98x0.95mm_HandSolder, symbol Device:R
- J10, J9: footprint Connector_PinHeader_2.54mm:PinHeader_1x04_P2.54mm_Vertical -> Connector_PinHeader_2.54mm:PinHeader_1x04_P2.54mm_Horizontal
- R18: value 1K -> 10k; LCSC (none) -> C25804
Connections:
- net +5P: now also R26.2
- net GND: now also R18.1, C29.2
- net LED_GREEN renamed AU_STATUS
- net AU_STATUS: now also C29.1, R26.1
Other:
- note added: "AU Status"
- note added: "LED status"
- note removed: "Blink=Ready"
- note removed: "LED statut"
- moved on the sheet: D8, R19

Commit message: fin du routage carte PAMI 2025
Parts:
- added J20: Conn_01x03, Connector_PinHeader_2.54mm:PinHeader_1x03_P2.54mm_Vertical, symbol Connector_Generic:Conn_01x03
- J5: now not fitted; now left out of the parts list
- J6: now fitted
Connections:
- net +5L: now also J20.2 (Pin_2)
- net GND: now also J20.1 (Pin_1)
- net LED_RED: now also U3.18 (IO10); no longer U3.38 (IO2)
- net M1_DIAG/uSW1: now also U3.8 (IO15); no longer U3.24 (IO47)
- net M2_DIAG/uSW2: now also U3.38 (IO2); no longer U3.8 (IO15)
- net TX_LIDAR: now also U3.24 (IO47); no longer U3.18 (IO10)
- net WS_5: now reaches D10.2 (DOUT)
- net WS_5: now also J20.3 (Pin_3)
- no-connect marks 27 -> 26
Other:
- moved on the sheet: JP10, JP11, JP8, JP9

Commit message: modification de bouton et fichier de prod
Parts:
- added R27: 31.6k, Resistor_SMD:R_0603_1608Metric_Pad0.98x0.95mm_HandSolder, symbol Device:R
- added SW5, SW6, SW7: SW_Push, SW_Push_1TS009xxxx-xxxx-xxxx_6x6x5mm, symbol Switch:SW_Push
- C1, C10, C13, C16, C17, C18, C19, C20, C21, C25, C26, C27, C28, C29, C3, C5, C6, C7, C8, C9: LCSC (none) -> C14663
- C12, C24, C4: LCSC C1588 -> C440198; Mouser (none) -> 81-GRM21BR61H106KE3L
- C2: Mouser (none) -> 81-GRM21BR61H106KE3L
- D1: value LED -> LED yellow; LCSC (none) -> C2290; Mouser (none) -> 710-150060YS75000
- D2, D6: Mouser (none) -> 621-1N4148W-F
- D3: value LED -> LED green; LCSC (none) -> C2290; Mouser (none) -> 710-150060VS75000
- D8: value LED -> LED red; LCSC (none) -> C2286
- J15, J7: now left out of the parts list
- J4: Mouser (none) -> 710-65100516121
- JP10, JP8: now not fitted
- Q1, Q2: Mouser (none) -> 621-DMG2302UK-7
- R1, R17, R19, R9: value 1K -> 1k
- R10, R11, R12, R13, R14, R20, R21, R22, R23, R24, R25: value 10K -> 10k; LCSC (none) -> C25804
- R15, R4: LCSC (none) -> C23182; Mouser (none) -> 603-RC0603FR-1068RL
- R2, R3, R6, R7: LCSC (none) -> C25804; now not fitted; now left out of the parts list
- SW2, SW3, SW4: Mouser (none) -> 710-431181015816; now not fitted; now left out of the parts list
- U1: Mouser (none) -> 926-LM1117MPX3.3NOPB; now not fitted
- U3: Mouser ESP32-S3-WROOM-1-N16R8 -> (none)
Connections:
- net BOOT0: now also SW5.1
- net COLORSIDE: now also SW7.1
- net ESP32_EN: now also SW6.1
- net GND: now also SW5.2, SW6.2, SW7.2
- no-connect marks 26 -> 28
Other:
- note added: "fermer les 2 JP (16 micro-pas)"
- note added: "mettre les resistances a chaque bout de la carte"
- note added: "sur la carte Batt R28=31,6k =>3.3V (R28=32,5k =>3.4V)"
- note added: "utilise 2 header 8p: wurth 61300811821"
- note removed: "sur la carte batt R28=32,5k =>3.4V R28=31,6k =>3.3V"
